Commit message: Update combined2.urdf.xacro

File: catkin_ws/src/robomuse/urdf/robomuse_base/combined2.urdf.xacro (robot description, xacro)
@@ -26,6 +26,6 @@
   <property name="base_size_z" value="0.005"/>
   <property name="base_mass" value="22.0"/>
-  <property name="caster_offset_x" value="0.27907"/>
-  <property name="caster_offset_y" value="0.2"/>
+  <property name="caster_offset_x" value="0.22"/>
+  <property name="caster_offset_y" value="0.28"/>
   <property name="caster_offset_z" value="0"/>
   <property name="caster_mass" value="0.1"/>
@@ -78,5 +78,5 @@
       </inertial>
       <visual>
-        <origin xyz="0 0 0.3" rpy="0 0 0"/>
+        <origin xyz="0 0 0.3" rpy="0 0 ${-M_PI/2}"/>
                 <geometry>
   			<mesh filename="package://robomuse/meshes/basenew.dae" />
@@ -85,5 +85,5 @@
       </visual>
       <collision>
-        <origin xyz="0 0 0.3" rpy="0 0 0"/>
+        <origin xyz="0 0 0.3" rpy="0 0 ${-M_PI/2}"/>
         	<geometry>
          		<mesh filename="package://robomuse/meshes/basenew.dae" />
@@ -92,5 +92,5 @@
     </link>
       <joint name="chassis_joint_base" type="fixed">
-      <origin xyz="0 .68 ${-0.26}" rpy="0 0 0"/>
+      <origin xyz=" .68 0 ${-0.26}" rpy="0 0 0"/>
       <child link="chassis_link"/>
       <parent link="base_link"/>
@@ -103,5 +103,5 @@
       </inertial>
       <visual>
-        <origin xyz="0 0 0" rpy="3.14 0 0"/>
+        <origin xyz="0 0 0" rpy="3.14 0 ${-M_PI/2}"/>
                 <geometry>
   			<mesh filename="package://robomuse/meshes/chassis.dae" />
@@ -110,5 +110,5 @@
       </visual>
       <collision>
-        <origin xyz="0 0 0" rpy="3.14 0 0"/>
+        <origin xyz="0 0 0" rpy="3.14 0 ${-M_PI/2}"/>
         	<geometry>
          		<mesh filename="package://robomuse/meshes/chassis.dae" />
@@ -148,7 +148,6 @@
       </inertial>
       <visual>
-        <origin xyz="0 0 0" rpy="${M_PI/2} 0 ${M_PI/2}"/>
-        <geometry>
-	      <!--mesh filename="package://youbot_description/meshes/youbot_base/front-left_wheel.dae" /-->
+        <origin xyz="0 0 0" rpy="${M_PI/2} 0 0"/>
+        <geometry>
           <cylinder radius="${wheel_radius}" length="${wheel_radius}"/>
         </geometry>
@@ -156,5 +155,5 @@
       </visual>
       <collision>
-        <origin xyz="0 0 0" rpy="${M_PI/2} 0 ${M_PI/2}"/>
+        <origin xyz="0 0 0" rpy="${M_PI/2} 0 0"/>
         <geometry>
           <cylinder radius="${wheel_radius}" length="${wheel_radius}"/>
@@ -164,5 +163,5 @@
 <!--fr-->
 	    <joint name="caster_joint_fr" type="continuous">
-      <origin xyz="${caster_offset_x} ${-caster_offset_y} ${caster_offset_z}" rpy="0 0 0"/>
+      <origin xyz="${-caster_offset_x} ${caster_offset_y} ${caster_offset_z}" rpy="0 0 0"/>
       <axis xyz="0 0 1"/>
       <limit effort="${caster_joint_effort}" velocity="${caster_joint_velocity}"/>
@@ -195,13 +194,12 @@
       </inertial>
       <visual>
-        <origin xyz="0 0 0" rpy="${M_PI/2} 0 ${M_PI/2}"/>
-        <geometry>
-          <!--mesh filename="package://youbot_description/meshes/youbot_base/front-right_wheel.dae" /-->
-          <cylinder radius="${wheel_radius}" length="${wheel_radius}"/>
-        </geometry>
-        <material name="Orange"/>
-      </visual>
-      <collision>
-        <origin xyz="0 0 0" rpy="${M_PI/2} 0 ${M_PI/2}"/>
+        <origin xyz="0 0 0" rpy="${M_PI/2} 0 0"/>
+        <geometry>
+             <cylinder radius="${wheel_radius}" length="${wheel_radius}"/>
+        </geometry>
+        <material name="Orange"/>
+      </visual>
+      <collision>
+        <origin xyz="0 0 0" rpy="${M_PI/2} 0 0"/>
         <geometry>
           <cylinder radius="${wheel_radius}" length="${wheel_radius}"/>
@@ -244,18 +242,17 @@
         <origin xyz="0 0 0" rpy="${M_PI/2} 0 ${M_PI/2}"/>
         <geometry>
-	      <!--mesh filename="package://youbot_description/meshes/youbot_base/front-left_wheel.dae" /-->
+	   <sphere radius="${wheel_radius/4*3}"/>
+        </geometry>
+        <material name="Orange"/>
+      </visual>
+      <collision>
+        <origin xyz="0 0 0" rpy="${M_PI/2} 0 ${M_PI/2}"/>
+        <geometry>
           <sphere radius="${wheel_radius/4*3}"/>
         </geometry>
-        <material name="Orange"/>
-      </visual>
-      <collision>
-        <origin xyz="0 0 0" rpy="${M_PI/2} 0 ${M_PI/2}"/>
-        <geometry>
-          <sphere radius="${wheel_radius/4*3}"/>
-        </geometry>
       </collision>
     </link>
       <joint name="rack_joint_base" type="fixed">
-      <origin xyz="${vertical_offset_x} ${vertical_offset_y - .20} 0" rpy="0 0 0"/>
+      <origin xyz="${vertical_offset_y - .20} ${vertical_offset_x} 0" rpy="0 0 0"/>
       <child link="rack_vertical_link1"/>
       <parent link="base_link"/>
@@ -282,5 +279,5 @@
     </link>
 <joint name="rack_joint_base1" type="fixed">
-      <origin xyz="${vertical_offset_x} ${-vertical_offset_y - .20} 0" rpy="0 0 0"/>
+      <origin xyz="${-vertical_offset_y - .2} ${vertical_offset_x - 0.025} 0" rpy="0 0 0"/>
       <child link="rack_vertical_link2"/>
       <parent link="base_link"/>
@@ -307,5 +304,5 @@
     </link>
 <joint name="rack_joint_base2" type="fixed">
-      <origin xyz="${-vertical_offset_x} ${-vertical_offset_y - .20} 0" rpy="0 0 0"/>
+      <origin xyz="${-vertical_offset_y - .23} ${-vertical_offset_x} 0" rpy="0 0 0"/>
       <child link="rack_vertical_link3"/>
       <parent link="base_link"/>
@@ -332,5 +329,5 @@
     </link>
 <joint name="rack_joint_base3" type="fixed">
-      <origin xyz="${-vertical_offset_x} ${vertical_offset_y - .20} 0" rpy="0 0 0"/>
+      <origin xyz="${-vertical_offset_y -0.03} ${-vertical_offset_x + 0.025} 0" rpy="0 0 0"/>
       <child link="rack_vertical_link4"/>
       <parent link="base_link"/>
@@ -357,5 +354,5 @@
     </link>
 <joint name="rack_joint_link11" type="fixed">
-      <origin xyz="${vertical_offset_x} ${vertical_offset_y} 0.090" rpy="0 0 0"/>
+      <origin xyz="${vertical_offset_x + 0.13} -0.035 0.090" rpy="0 0 0"/>
       <child link="rack_link2"/>
       <parent link="rack_vertical_link1"/>
@@ -368,5 +365,5 @@
       </inertial>
       <visual>
-        <origin xyz="${-rack_base_size_x} ${-rack_base_size_y} 0.09" rpy="0 0 0"/>
+        <origin xyz="${-rack_base_size_x} ${-rack_base_size_y} 0.09" rpy="0 0 ${M_PI/2}"/>
                 <geometry>
           <box size="${rack_base_size_x} ${rack_base_size_y} ${rack_base_size_z}"/>
@@ -375,5 +372,5 @@
       </visual>
       <collision>
-        <origin xyz="${-rack_base_size_x} ${-rack_base_size_y} 0.09" rpy="0 0 0"/>
+        <origin xyz="${-rack_base_size_x} ${-rack_base_size_y} 0.09" rpy="0 0 ${M_PI/2}"/>
         <geometry>
           <box size="${rack_base_size_x} ${rack_base_size_y} ${rack_base_size_z}"/>
@@ -382,5 +379,5 @@
 </link>
 <joint name="rack_joint_link21" type="fixed">
-      <origin xyz="${vertical_offset_x} ${vertical_offset_y} 0.190" rpy="0 0 0"/>
+      <origin xyz="${vertical_offset_x + 0.13} -0.035 0.190" rpy="0 0 0"/>
       <child link="rack_link3"/>
       <parent link="rack_vertical_link1"/>
@@ -393,5 +390,5 @@
       </inertial>
       <visual>
-        <origin xyz="${-rack_base_size_x} ${-rack_base_size_y} 0.19" rpy="0 0 0"/>
+        <origin xyz="${-rack_base_size_x} ${-rack_base_size_y} 0.19" rpy="0 0 ${M_PI/2}"/>
                 <geometry>
           <box size="${rack_base_size_x} ${rack_base_size_y} ${rack_base_size_z}"/>
@@ -400,5 +397,5 @@
       </visual>
       <collision>
-        <origin xyz="${-rack_base_size_x} ${-rack_base_size_y} 0.19" rpy="0 0 0"/>
+        <origin xyz="${-rack_base_size_x} ${-rack_base_size_y} 0.19" rpy="0 0 ${M_PI/2}"/>
         <geometry>
           <box size="${rack_base_size_x} ${rack_base_size_y} ${rack_base_size_z}"/>
@@ -407,5 +404,5 @@
 </link>
 <joint name="rack_joint_link31" type="fixed">
-      <origin xyz="${vertical_offset_x} ${vertical_offset_y} 0.290" rpy="0 0 0"/>
+      <origin xyz="${vertical_offset_x + 0.13} -0.035 0.290" rpy="0 0 0"/>
       <child link="rack_link4"/>
       <parent link="rack_vertical_link1"/>
@@ -417,5 +414,5 @@
         <inertia ixx="0.00774243378" ixy="-0.01404395602" ixz="-.00042131868" iyy="0.04530596321" iyz="0.00017409863" izz="0.05303446911"/>      </inertial>
       <visual>
-        <origin xyz="${-rack_base_size_x} ${-rack_base_size_y} 0.29" rpy="0 0 0"/>
+        <origin xyz="${-rack_base_size_x} ${-rack_base_size_y} 0.29" rpy="0 0 ${M_PI/2}"/>
                 <geometry>
           <box size="${rack_base_size_x} ${rack_base_size_y} ${rack_base_size_z}"/>
@@ -424,5 +421,5 @@
       </visual>
       <collision>
-        <origin xyz="${-rack_base_size_x} ${-rack_base_size_y} 0.29" rpy="0 0 0"/>
+        <origin xyz="${-rack_base_size_x} ${-rack_base_size_y} 0.29" rpy="0 0 ${M_PI/2}"/>
         <geometry>
           <box size="${rack_base_size_x} ${rack_base_size_y} ${rack_base_size_z}"/>
@@ -431,5 +428,5 @@
 </link>
 <joint name="rack_joint_link41" type="fixed">
-      <origin xyz="${vertical_offset_x} ${vertical_offset_y} 0.390" rpy="0 0 0"/>
+      <origin xyz="${vertical_offset_x + 0.13} -0.035 0.390" rpy="0 0 0"/>
       <child link="rack_link5"/>
       <parent link="rack_vertical_link1"/>
@@ -441,5 +438,5 @@
         <inertia ixx="0.00774243378" ixy="-0.01404395602" ixz="-.00042131868" iyy="0.04530596321" iyz="0.00017409863" izz="0.05303446911"/>      </inertial>
       <visual>
-        <origin xyz="${-rack_base_size_x} ${-rack_base_size_y} 0.39" rpy="0 0 0"/>
+        <origin xyz="${-rack_base_size_x} ${-rack_base_size_y} 0.39" rpy="0 0 ${M_PI/2}"/>
                 <geometry>
           <box size="${rack_base_size_x} ${rack_base_size_y} ${rack_base_size_z}"/>
@@ -448,5 +445,5 @@
       </visual>
       <collision>
-        <origin xyz="${-rack_base_size_x} ${-rack_base_size_y} 0.39" rpy="0 0 0"/>
+        <origin xyz="${-rack_base_size_x} ${-rack_base_size_y} 0.39" rpy="0 0 ${M_PI/2}"/>
         <geometry>
           <box size="${rack_base_size_x} ${rack_base_size_y} ${rack_base_size_z}"/>
@@ -455,5 +452,6 @@
 </link>
  <joint name="camera_rgb_joint" type="fixed">
-      <origin xyz="0 0.3 0.1" rpy="0 0 ${M_PI/2} "/>
+      <!--origin xyz="0 0.3 0.1" rpy="0 0 ${M_PI/2} "/-->
+      <origin xyz="0 -.03 0.1" rpy="0 0 0 "/>
       <parent link="base_link"/>
       <child link="camera_rgb_frame" />
@@ -461,5 +459,5 @@
     <link name="camera_rgb_frame"/>
     <joint name="camera_rgb_optical_joint" type="fixed">
-      <origin xyz="0 0 0" rpy="${-M_PI/2} 0 ${-M_PI/2}" />
+      <origin xyz="0 0 0" rpy="${-M_PI/2} 0 0" />
       <parent link="camera_rgb_frame" />
       <child link="camera_rgb_optical_frame" />
@@ -473,5 +471,5 @@
       <link name="camera_link">
       <visual>
-       <origin xyz="0 0 0" rpy="0 0 ${M_PI/2}"/>
+       <origin xyz="0 0 0" rpy="0 0 0"/>
         <geometry>
          <mesh filename="package://robomuse/meshes/kinect.dae"/>
@@ -481,5 +479,5 @@
         <origin xyz="0.0 0.0 0.0" rpy="0 0 0"/>
   	    <geometry>
-  	      <box size="0.07271 0.27794 0.073"/>
+  	       <mesh filename="package://robomuse/meshes/kinect.dae"/>
   	    </geometry>
   	  </collision>
